File: hardware/6_bay_charg/LEDs_driver.kicad_sch (KiCad schematic)
At the start: 19 parts, among them IC1 PCA9634PW

Commit message: Integrate fan, USB interface, firmware, and cleaned KiCad schematics
- Added 12V fan for thermal management
- Integrated USB interface (hardware and firmware)
- Added initial firmware implementation
- Cleaned and refactored KiCad schematics
- Updated and regenerated schematic PDF plots
- Updated project README to reflect latest architecture
Connections:
- net 3.3V renamed +3.3V
Other:
- note added: "LED driver"
- moved on the sheet: C21, C22, D10, D3, D4, D5, D6, D7, D8, D9, IC1, R14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
